File: Hardware/PCB_OpenBook.brd (EAGLE design)
At the start: 170.2 x 111.2 mm, 103 parts, among them IC1 XC6220A331MR-G, IC4 XC6220A331MR-G, J1 FH34SRJ-24S-0.5SH_99_, J2 SAMACSYS_PARTS_USB4110-GF-A, J3 QWIIC_RIGHT_ANGLE, J4 112A-TAAR-R03_ATTEND, Q1 20V/4.2A/52mΩ/1.4W, Q2 20V/4.2A/52mΩ/1.4W, Q3 SI1308EDL-T1-GE3, U1 W25Q512JVEIQ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

Commit message: Update PCB
Parts:
- moved TP11 88.0 mm to (93.1, 1.06)
- moved TP12 66.3 mm to (96.6, 8.51)
- moved TP6 13.2 mm to (16.3, 89.6)
- moved R2-USB1 11.9 mm to (153.7, 40.3), turned to 0 degrees
- moved EPD_C12 6.19 mm to (73.0, 3.45), turned to 270 degrees
- moved TP4 5.15 mm to (40.2, 89.5)
- moved TP16 4.48 mm to (166.2, 16.0)
- moved EPD_C1 4.28 mm to (91.9, 11.4), turned to 90 degrees
- moved R3 3.46 mm to (67.1, 2.13)
- moved EPD_C8 3.32 mm to (81.4, 11.4)
- moved EPD_C9 3.15 mm to (79.7, 11.4)
- moved EPD_C11 2.80 mm to (76.1, 11.3)
- moved EPD_C10 2.79 mm to (78.0, 11.4)
- moved TP10 2.65 mm to (125.3, 6.51)
- moved C1_BAT1 2.50 mm to (118.4, 31.3)
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Connections:
- removed net N$22: EPD_C2.2, J1.5
- new net N$17: EPD_C1.1, J1.4
- net 3V3: now also R1.1, R_BOOT.1, R_CHANGE.1, R_CL1.1, R_RESET.1; no longer R1.2, R_BOOT.2, R_CHANGE.2, R_CL1.2, R_RESET.2
- net EPD_3V3_C: now also R_CL1.2; no longer R_CL1.1
- net GDR: now also R4.1; no longer R4.2
- net GND: now also EPD_C1.2, EPD_C10.2, EPD_C11.2, EPD_C12.2, EPD_C2.2, EPD_C5.2, EPD_C6.2, EPD_C7.2, EPD_C8.2, EPD_C9.2, R4.2; no longer EPD_C1.1, EPD_C10.1, EPD_C11.1, EPD_C12.1, EPD_C2.1, EPD_C5.1, EPD_C6.1, EPD_C7.1, EPD_C8.1, EPD_C9.1, R4.1
- net GPIO8: now also R1.2; no longer R1.1
- net IO/BOOT: now also R_BOOT.2; no longer R_BOOT.1
- net IO/CHANGE: now also R_CHANGE.2; no longer R_CHANGE.1
- net N$10: now also R1_BAT.1; no longer R1_BAT.2
- net N$11: now also R1_BAT.2; no longer R1_BAT.1
- net N$13: now also EPD_C10.1; no longer EPD_C10.2
- net N$14: now also R_CAPACITOR.2; no longer R_CAPACITOR.1
- net N$15: now also EPD_C8.1; no longer EPD_C8.2
- net N$16: now also EPD_C7.1; no longer EPD_C7.2
- net N$18: now also R_RESET.2; no longer R_RESET.1
- net N$19: now also EPD_C6.1; no longer EPD_C6.2
- net N$20: now also EPD_C2.1, J1.5; no longer EPD_C1.2, J1.4
- net N$21: now also EPD_C5.1; no longer EPD_C5.2
- net N$9: now also EPD_C12.1; no longer EPD_C12.2
- net PREVGL: now also EPD_C11.1, EPD_C9.1; no longer EPD_C11.2, EPD_C9.2
- net RESE: now also R3.1; no longer R3.2
- net RESE': now also R3.2; no longer R3.1
- net VRTC: now also R_CAPACITOR.1; no longer R_CAPACITOR.2
Routing:
- net GND: track 681.1 -> 774.4 mm, vias 24 -> 39
- net EPD_RST: track 139.1 -> 102.8 mm, vias 3 -> 5
- net N$20: track 6.61 -> 41.8 mm, vias 0 -> 2
- net N$22: track 31.9 -> 0.00 mm, vias 2 -> 0
- net RESET: track 70.8 -> 96.1 mm
- net I2C_PW: track 163.7 -> 188.3 mm
- net SCL: track 228.7 -> 207.3 mm
- net SDA: track 237.6 -> 219.2 mm, vias 6 -> 5
- net EPD_3V3: track 273.5 -> 290.7 mm
- net 32KHZ: track 92.7 -> 107.5 mm, vias 4 -> 6
- net N$2: track 20.7 -> 32.4 mm, vias 2 -> 0
- net SCK: track 206.3 -> 216.0 mm, vias 9 -> 10
- net EPD_DC: track 92.5 -> 102.1 mm
- net N$17: track 0.00 -> 7.11 mm
- net FLASH_CS: track 139.2 -> 132.7 mm, vias 6 -> 8
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