File: Hardware/PCB_OpenBook.brd (EAGLE design)
At the start: 170.2 x 111.2 mm, 103 parts, among them IC1 XC6220A331MR-G, IC4 XC6220A331MR-G, J1 FH34SRJ-24S-0.5SH_99_, J2 SAMACSYS_PARTS_USB4110-GF-A, J3 QWIIC_RIGHT_ANGLE, J4 112A-TAAR-R03_ATTEND, Q1 20V/4.2A/52mΩ/1.4W, Q2 20V/4.2A/52mΩ/1.4W, Q3 SI1308EDL-T1-GE3, U1 W25Q512JVEIQ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

Commit message: Update PCB
Routing:
- net GND: vias 39 -> 45
Changed lines of the file:
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@@
 <attribute name="VALUE" x="7.9262" y="75.385" size="0.635" layer="27" align="center"/>
 </element>
-<element uuid="2882400010" name="L1" library="DeskAssistant v19 v1" library_urn="urn:adsk.wipprod:fs.file:vf.UKByVhMZT-yf0EmZIsR-pg" package="IND_4828-WE-TPC_WRE" package3d_urn="urn:adsk.eagle:package:47550349/1" value="68uH" x="79.71" y="21.52" smashed="yes" rot="R270">
+<element uuid="2882400010" name="L1" library="DeskAssistant v19 v1" library_urn="urn:adsk.wipprod:fs.file:vf.UKByVhMZT-yf0EmZIsR-pg" package="IND_4828-WE-TPC_WRE" package3d_urn="urn:adsk.eagle:package:47550349/1" override_locally_modified="yes" value="68uH" x="79.71" y="21.52" smashed="yes" rot="R270">
 <attribute name="COPYRIGHT" value="Copyright (C) 2024 Ultra Librarian. All rights reserved." x="60.66" y="-28.01" size="1.778" layer="27" rot="R270" display="off"/>
 <attribute name="MANUFACTURER_PART_NUMBER" value="744043680" x="60.66" y="-28.01" size="1.778" layer="27" rot="R270" display="off"/>
@@
 </element>
 <element name="TP1" library="DeskAssistant v19 v1" library_urn="urn:adsk.wipprod:fs.file:vf.UKByVhMZT-yf0EmZIsR-pg" package="TP20R" package3d_urn="urn:adsk.eagle:package:47550340/1" value="TPTP20R" x="3.14" y="59.36" smashed="yes">
+<attribute name="3D_NAME" value="TX" x="3.14" y="59.36" size="1.778" layer="27" display="off"/>
 <attribute name="NAME" x="2.14" y="60.41" size="0.635" layer="25"/>
 <attribute name="POPULARITY" value="2" x="95.85" y="-33.35" size="1.778" layer="27" display="off"/>
@@
 <wire x1="14.61175" y1="44.94325" x2="14.57" y2="44.925" width="0.15" layer="1"/>
 <wire x1="14.61175" y1="46.1205" x2="14.57" y2="46.175" width="0.15" layer="1"/>
-<wire x1="37.87975" y1="48.0595" x2="35.94075" y2="48.0595" width="0.15" layer="1"/>
-<wire x1="39.7495" y1="49.92925" x2="37.87975" y2="48.0595" width="0.15" layer="1"/>
+<wire x1="35.94075" y1="48.0595" x2="37.87975" y2="48.0595" width="0.15" layer="1"/>
+<wire x1="37.87975" y1="48.0595" x2="39.7495" y2="49.92925" width="0.15" layer="1"/>
 <wire x1="35.94075" y1="48.0595" x2="35.905" y2="48.045" width="0.15" layer="1"/>
 <wire x1="39.7495" y1="49.92925" x2="39.8" y2="49.95" width="0.15" layer="1"/>
@@
 <via x="165.5" y="3.55" extent="1-16" drill="0.35" alwaysstop="yes">
 </via>
+<via x="15.9" y="41.4" extent="1-16" drill="0.35" alwaysstop="yes">
+</via>
+<via x="21.15" y="39.4" extent="1-16" drill="0.35" alwaysstop="yes">
+</via>
+<via x="21.5" y="35.1" extent="1-16" drill="0.35" alwaysstop="yes">
+</via>
+<via x="16.1" y="35.6" extent="1-16" drill="0.35" alwaysstop="yes">
+</via>
+<via x="5.1" y="61.25" extent="1-16" drill="0.35" alwaysstop="yes">
+</via>
+<via x="19.75" y="49.55" extent="1-16" drill="0.35" alwaysstop="yes">
+</via>
 </signal>
 <signal name="N$1">
@@
 <wire x1="58.93175" y1="45.91275" x2="62.11725" y2="49.09825" width="0.15" layer="16"/>
 <wire x1="34.55575" y1="45.91275" x2="58.93175" y2="45.91275" width="0.15" layer="16"/>
-<wire x1="32.2705" y1="43.6275" x2="34.55575" y2="45.91275" width="0.15" layer="1"/>
+<wire x1="34.55575" y1="45.91275" x2="32.2705" y2="43.6275" width="0.15" layer="1"/>
 <wire x1="30.0545" y1="43.6275" x2="32.2705" y2="43.6275" width="0.15" layer="16"/>
 <wire x1="27.8385" y1="41.4115" x2="30.0545" y2="43.6275" width="0.15" layer="16"/>
@@
 <wire x1="8.93325" y1="37.672" x2="8.93325" y2="37.2565" width="0.3" layer="1"/>
 <wire x1="19.2515" y1="31.78575" x2="19.3" y2="31.72" width="0.3" layer="1"/>
-<wire x1="8.93325" y1="37.672" x2="8.87" y2="37.68" width="0.3" layer="1"/>
+<wire x1="8.87" y1="37.68" x2="8.93325" y2="37.672" width="0.3" layer="1"/>
 <wire x1="9.141" y1="82.546" x2="9.141" y2="88.70925" width="0.3" layer="1"/>
 <wire x1="5.54" y1="78.945" x2="9.141" y2="82.546" width="0.3" layer="1"/>
@@
 <wire x1="38.01825" y1="52.42225" x2="37.8105" y2="52.2145" width="0.3" layer="1"/>
 <wire x1="43.0735" y1="52.42225" x2="38.01825" y2="52.42225" width="0.3" layer="1"/>
-<wire x1="43.6275" y1="51.86825" x2="43.0735" y2="52.42225" width="0.3" layer="1"/>
+<wire x1="43.0735" y1="52.42225" x2="43.6275" y2="51.86825" width="0.3" layer="1"/>
 <wire x1="35.94075" y1="49.37525" x2="35.905" y2="49.315" width="0.3" layer="1"/>
 <wire x1="43.6275" y1="51.86825" x2="43.695" y2="51.855" width="0.3" layer="1"/>
@@
 <wire x1="47.2285" y1="90.856" x2="43.14275" y2="86.77025" width="0.3" layer="1"/>
 <wire x1="43.14275" y1="52.56075" x2="43.0735" y2="52.42225" width="0.3" layer="1"/>
-<wire x1="47.2285" y1="90.856" x2="47.62" y2="90.88" width="0.3" layer="1"/>
+<wire x1="47.62" y1="90.88" x2="47.2285" y2="90.856" width="0.3" layer="1"/>
 <wire x1="13.64225" y1="88.7785" x2="9.2795" y2="88.7785" width="0.3" layer="1"/>
 <wire x1="21.39825" y1="96.5345" x2="13.64225" y2="88.7785" width="0.3" layer="1"/>
@@
 <wire x1="5.60925" y1="78.8065" x2="6.7865" y2="77.62925" width="0.3" layer="1"/>
 <wire x1="8.79475" y1="37.8105" x2="8.87" y2="37.68" width="0.3" layer="1"/>
-<wire x1="5.60925" y1="78.8065" x2="4.8762" y2="78.93" width="0.3" layer="1"/>
+<wire x1="4.8762" y1="78.93" x2="5.60925" y2="78.8065" width="0.3" layer="1"/>
 <wire x1="165.43825" y1="8.4485" x2="165.02275" y2="8.4485" width="0.3" layer="1"/>
 <wire x1="166.2" y1="9.21025" x2="165.43825" y2="8.4485" width="0.3" layer="1"/>
@@
 <wire x1="75.621" y1="16.2045" x2="58.3085" y2="16.2045" width="0.3" layer="1"/>
 <wire x1="19.39" y1="31.64725" x2="19.3" y2="31.72" width="0.3" layer="1"/>
-<wire x1="75.621" y1="16.2045" x2="75.73" y2="16.15" width="0.3" layer="1"/>
+<wire x1="75.73" y1="16.15" x2="75.621" y2="16.2045" width="0.3" layer="1"/>
 </signal>
 <signal name="N$3">
@@
 <wire x1="8.93325" y1="55.123" x2="8.93325" y2="54.846" width="0.15" layer="1"/>
 <wire x1="35.94075" y1="50.62175" x2="35.905" y2="50.585" width="0.15" layer="1"/>
-<wire x1="8.93325" y1="55.123" x2="8.87" y2="55.18" width="0.15" layer="1"/>
+<wire x1="8.87" y1="55.18" x2="8.93325" y2="55.123" width="0.15" layer="1"/>
 <wire x1="94.80325" y1="17.24325" x2="110.1075" y2="1.939" width="0.15" layer="1"/>
 <wire x1="94.80325" y1="18.1435" x2="94.80325" y2="17.24325" width="0.15" layer="16"/>
@@
 <wire x1="5.54" y1="76.729" x2="6.2325" y2="76.0365" width="0.15" layer="1"/>
 <wire x1="11.357" y1="37.74125" x2="11.41" y2="37.68" width="0.15" layer="1"/>
-<wire x1="5.54" y1="76.729" x2="5.4762" y2="76.73" width="0.15" layer="1"/>
+<wire x1="5.4762" y1="76.73" x2="5.54" y2="76.729" width="0.15" layer="1"/>
 <wire x1="124.7885" y1="-3.047" x2="129.7745" y2="-3.047" width="0.15" layer="16"/>
 <wire x1="124.2345" y1="-3.601" x2="124.7885" y2="-3.047" width="0.15" layer="16"/>
@@
 <wire x1="35.282875" y1="41.238375" x2="42.03475" y2="47.99025" width="0.15" layer="1"/>
 <wire x1="18.21275" y1="40.92675" x2="34.97125" y2="40.92675" width="0.15" layer="16"/>
-<wire x1="15.235" y1="37.949" x2="18.21275" y2="40.92675" width="0.15" layer="1"/>
-<wire x1="15.235" y1="37.74125" x2="15.235" y2="37.949" width="0.15" layer="1"/>
+<wire x1="18.21275" y1="40.92675" x2="15.235" y2="37.949" width="0.15" layer="1"/>
+<wire x1="15.235" y1="37.949" x2="15.235" y2="37.74125" width="0.15" layer="1"/>
 <wire x1="43.6275" y1="47.99025" x2="43.695" y2="48.045" width="0.15" layer="1"/>
 <wire x1="15.235" y1="37.74125" x2="15.22" y2="37.68" width="0.15" layer="1"/>
@@
 <wire x1="25.484" y1="41.4115" x2="29.98525" y2="45.91275" width="0.15" layer="16"/>
 <wire x1="25.0685" y1="41.4115" x2="25.484" y2="41.4115" width="0.15" layer="1"/>
-<wire x1="21.606" y1="37.949" x2="25.0685" y2="41.4115" width="0.15" layer="1"/>
-<wire x1="21.606" y1="37.74125" x2="21.606" y2="37.949" width="0.15" layer="1"/>
+<wire x1="25.0685" y1="41.4115" x2="21.606" y2="37.949" width="0.15" layer="1"/>
+<wire x1="21.606" y1="37.949" x2="21.606" y2="37.74125" width="0.15" layer="1"/>
 <wire x1="35.8715" y1="51.799" x2="35.905" y2="51.855" width="0.15" layer="1"/>
 <wire x1="21.606" y1="37.74125" x2="21.57" y2="37.68" width="0.15" layer="1"/>
@@
 <wire x1="19.59775" y1="75.7595" x2="19.59775" y2="64.1255" width="0.15" layer="1"/>
 <wire x1="12.742" y1="55.19225" x2="12.68" y2="55.18" width="0.15" layer="1"/>
-<wire x1="19.59775" y1="75.7595" x2="19.64" y2="75.79" width="0.15" layer="1"/>
+<wire x1="19.64" y1="75.79" x2="19.59775" y2="75.7595" width="0.15" layer="1"/>
 </signal>
 <signal name="RTC_RST">
@@
 <wire x1="19.2515" y1="33.03225" x2="19.2515" y2="37.46425" width="0.15" layer="1"/>
 <wire x1="19.2515" y1="37.46425" x2="19.04375" y2="37.672" width="0.15" layer="1"/>
-<wire x1="19.2515" y1="33.03225" x2="19.3" y2="33.02" width="0.15" layer="1"/>
+<wire x1="19.3" y1="33.02" x2="19.2515" y2="33.03225" width="0.15" layer="1"/>
 <wire x1="19.04375" y1="37.672" x2="19.03" y2="37.68" width="0.15" layer="1"/>
 </signal>
